Commit message: Local research changes + collected documentation
Adds documentation collected during personal research and any local
edits made on top of upstream. Docs in docs/ cover training pipeline,
reward tuning, standing policy research, hardware notes, and a
walkthrough for individuals training their own policies.

File: open_duck_reference_motion_generator/robots/open_duck_mini_v2/open_duck_mini_v2.urdf (robot description, URDF)
Before this commit: robot open_duck_mini_v2, 21 links, 20 joints
Links:
- removed link knee_and_ankle_assembly_4
- removed link left_antenna_holder
- removed link right_antenna_holder
- added link imu, mass 1e-9
- added link right_cache, mass 0.12407; collision mesh filename=package://assets/drive_palonier.stl; collision mesh filename=package://assets/left_knee_to_ankle_left_sheet.stl
- link foot_assembly: mass 0.075240000000000015201 -> 0.07524; geometry collision mesh filename=package://assets/foot_bottom_pla.stl; collision mesh filename=package://assets/foot_bottom_tpu.stl
- link foot_assembly_2: mass 0.075240000000000015201 -> 0.07524; geometry collision mesh filename=package://assets/foot_bottom_pla.stl; collision mesh filename=package://assets/foot_bottom_tpu.stl
- link head_assembly: mass 0.35258298534369525434 -> 0.406607; geometry collision mesh filename=package://assets/antenna.stl; collision mesh filename=package://assets/antenna.stl
- link head_pitch_to_yaw: mass 0.016937787992336000853 -> 0.0169378; geometry collision mesh filename=package://assets/head_pitch_to_yaw.stl; visual mesh filename=package://assets/head_pitch_to_yaw.stl
- link hip_roll_assembly: mass 0.066480000000000011307 -> 0.06648; geometry collision mesh filename=package://assets/drive_palonier.stl; collision mesh filename=package://assets/passive_palonier.stl
- link hip_roll_assembly_2: mass 0.066480000000000011307 -> 0.06648; geometry collision mesh filename=package://assets/drive_palonier.stl; collision mesh filename=package://assets/passive_palonier.stl
- link knee_and_ankle_assembly: mass 0.12407000000000001361 -> 0.12407; geometry collision mesh filename=package://assets/drive_palonier.stl; collision mesh filename=package://assets/left_cache.stl
- link knee_and_ankle_assembly_2: mass 0.072590000000000015623 -> 0.07259; geometry collision mesh filename=package://assets/drive_palonier.stl; collision mesh filename=package://assets/left_knee_to_ankle_left_sheet.stl
- link knee_and_ankle_assembly_3: mass 0.12407000000000004136 -> 0.07259; geometry collision mesh filename=package://assets/drive_palonier.stl; collision mesh filename=package://assets/left_knee_to_ankle_left_sheet.stl
- link left_roll_to_pitch_assembly: mass 0.075160000000000004583 -> 0.07516; geometry collision mesh filename=package://assets/drive_palonier.stl; collision mesh filename=package://assets/left_roll_to_pitch.stl
- link neck_pitch_assembly: mass 0.066180000000000016591 -> 0.06618; geometry collision mesh filename=package://assets/drive_palonier.stl; collision mesh filename=package://assets/neck_left_sheet.stl
- link neck_yaw_assembly: mass 0.091809888579250376051 -> 0.0918099; geometry collision mesh filename=package://assets/drive_palonier.stl; collision mesh filename=package://assets/head_yaw_to_roll.stl
- link right_roll_to_pitch_assembly: mass 0.075160000000000004583 -> 0.07516; geometry collision mesh filename=package://assets/drive_palonier.stl; collision mesh filename=package://assets/passive_palonier.stl
- link trunk_assembly: mass 0.69852641931996084512 -> 0.698526; geometry collision mesh filename=package://assets/battery_pack_lid.stl; collision mesh filename=package://assets/bms.stl
Joints:
- removed joint left_antenna
- removed joint right_antenna
- added joint imu_frame: type fixed, parent trunk_assembly, child imu, origin xyz=-0.08711 0 0.0422909 rpy=-0 0 -0, axis 0 0 0
- joint head_frame: origin xyz=0.04244999999999957141 2.135878279796443735e-17 0.035950000000000377487 rpy=-0 1.570796326794896558 0 -> xyz=0.04245 -0 0.03595 rpy=-0 1.5708 0
- joint head_pitch: limit lower=-0.785398163397448279 upper=0.785398163397448279 effort=100 velocity=100 -> lower=-0.785398 upper=0.785398 effort=10 velocity=10; origin xyz=-5.42101086242752217e-17 0.066000000000000086375 -1.0408340855860842566e-17 rpy=-1.9479487599482720301e-16 -1.1423136863502905442e-16 1.7347234747146296461e-18 -> xyz=-0 0.066 -0 rpy=-0 -0 0
- joint head_roll: limit lower=-0.52359877559829881566 upper=0.52359877559829881566 effort=100 velocity=100 -> lower=-0.523599 upper=0.523599 effort=10 velocity=10; origin xyz=0.040950000000000000289 -4.2214766838438722019e-16 -0.019149999999999833822 rpy=1.2411687278497551329e-14 -1.5707963267948830133 0 -> xyz=0.04095 0 -0.01915 rpy=-0 -1.5708 0
- joint head_yaw: limit lower=-2.7925268031909271649 upper=2.7925268031909271649 effort=100 velocity=100 -> lower=-2.79253 upper=2.79253 effort=10 velocity=10; origin xyz=-9.9746599868666407929e-18 0.056999999999999967359 0.019050000000000014838 rpy=-1.570796326794896558 -1.3706437208012195828e-25 6.1232339958582419871e-17 -> xyz=-0 0.057 0.01905 rpy=-1.5708 0 0
- joint left_ankle: limit lower=-1.570796326794896558 upper=1.570796326794896558 effort=100 velocity=100 -> lower=-1.5708 upper=1.5708 effort=10 velocity=10; origin xyz=-7.9103390504542403505e-16 -0.078649999999999428701 9.9999999999794697558e-05 rpy=1.636340693842024721e-16 1.1379785959205303308e-15 -2.7755597583208935156e-17 -> xyz=0 -0.07865 0.0001 rpy=0 0 0
- joint left_foot_frame: origin xyz=0.00049999999999995187183 -0.036224999999999729638 0.019550000000000331002 rpy=-1.570796326794896558 4.8789097652664912905e-18 2.353432088828639061e-23 -> xyz=0.0005 -0.036225 0.01955 rpy=-1.5708 -0 -0
- joint left_hip_pitch: limit lower=-1.2217304763960306069 upper=0.52359877559829881566 effort=100 velocity=100 -> lower=-1.22173 upper=0.523599 effort=10 velocity=10; origin xyz=0.074149999999999799405 -1.9529191631895148618e-17 0.035109999999999898235 rpy=3.141592653589793116 1.570796326794896336 0 -> xyz=0.07415 -0 0.03511 rpy=-3.14159 1.5708 0
- joint left_hip_roll: limit lower=-0.43633231299858238339 upper=0.43633231299858238339 effort=100 velocity=100 -> lower=-0.436332 upper=0.436332 effort=10 velocity=10; origin xyz=0.019050000000003588368 4.3576253716537394212e-15 -0.046015000000001519964 rpy=-1.5707963267949396347 9.7936145200150713608e-14 1.5707963267946445374 -> xyz=0.01905 0 -0.046015 rpy=-1.5708 0 1.5708
- joint left_hip_yaw: limit lower=-0.52359877559829881566 upper=0.52359877559829881566 effort=100 velocity=100 -> lower=-0.523599 upper=0.523599 effort=10 velocity=10; origin xyz=-0.018999999999998434808 0.035000000000000974776 0.04594093881237738819 rpy=-1.5205902553582758499e-16 -2.2037927038784495587e-14 -6.3658912806794774433e-27 -> xyz=-0.019 0.035 0.0459409 rpy=0 -0 -0
- joint left_knee: limit lower=-1.570796326794896558 upper=1.570796326794896558 effort=100 velocity=100 -> lower=-1.5708 upper=1.5708 effort=10 velocity=10; origin xyz=-2.9837243786801082024e-16 -0.078650000000000871991 9.99999999999751088e-05 rpy=-2.6413758326899544516e-16 -7.0075679691128679348e-24 -2.4877517507049828295e-26 -> xyz=-0 -0.07865 0.0001 rpy=-0 0 -0
- joint neck_pitch: limit lower=-0.34906585039886589561 upper=1.1344640137963142301 effort=100 velocity=100 -> lower=-0.349066 upper=1.13446 effort=10 velocity=10; origin xyz=0.00099999999999899474856 0.019150000000000326483 0.090000938812376224396 rpy=1.57079632679489678 -2.2204460492503130808e-14 6.1232449680326617825e-17 -> xyz=0.001 0.01915 0.0900009 rpy=1.5708 -0 0
- joint right_ankle: limit lower=-1.570796326794896558 upper=1.570796326794896558 effort=100 velocity=100 -> lower=-1.5708 upper=1.5708 effort=10 velocity=10; origin xyz=1.3877787807814456755e-17 -0.078649999999999928302 0.00010000000000004449774 rpy=-2.6413812280837946538e-16 -1.7764738567684265366e-22 4.6805027693161558698e-25 -> xyz=-0.07865 -0 0.0001 rpy=0 0 0; parent knee_and_ankle_assembly_4 -> knee_and_ankle_assembly_3
- joint right_foot_frame: origin xyz=0.00050000000000022942759 -0.036224999999999812905 0.019550000000000553046 rpy=-1.570796326794896558 -2.2055201956572090666e-25 -2.8950564132886956449e-25 -> xyz=-0.036225 0.0005 0.01735 rpy=1.5708 0 1.5708
- joint right_hip_pitch: child knee_and_ankle_assembly_3 -> right_cache; limit lower=-0.52359877559829881566 upper=1.2217304763960306069 effort=100 velocity=100 -> lower=-0.523599 upper=1.22173 effort=10 velocity=10; origin xyz=-0.074149999999999771649 5.1732706660145844069e-16 0.035110000000000037013 rpy=-6.1899281068357555747e-22 1.570796326794896336 0 -> xyz=-0.07415 0 0.03511 rpy=-0 1.5708 0
- joint right_hip_roll: limit lower=-0.43633231299858238339 upper=0.43633231299858238339 effort=100 velocity=100 -> lower=-0.436332 upper=0.436332 effort=10 velocity=10; origin xyz=0.019050000000008570494 4.0564773762241657096e-14 -0.046015000000004170622 rpy=-1.5707963267947786523 -8.9077711856609251111e-14 1.5707963267946440933 -> xyz=0.01905 0 -0.046015 rpy=-1.5708 -0 1.5708
- joint right_hip_yaw: limit lower=-0.52359877559829881566 upper=0.52359877559829881566 effort=100 velocity=100 -> lower=-0.523599 upper=0.523599 effort=10 velocity=10; origin xyz=-0.018999999999998431338 -0.03500000000000151601 0.045940938812377415945 rpy=-5.7327222785292536251e-16 -2.1926904736366604217e-14 -2.7755575616618406396e-16 -> xyz=-0.019 -0.035 0.0459409 rpy=-0 -0 -0
- joint right_knee: child knee_and_ankle_assembly_4 -> knee_and_ankle_assembly_3; limit lower=-1.570796326794896558 upper=1.570796326794896558 effort=100 velocity=100 -> lower=-1.5708 upper=1.5708 effort=10 velocity=10; origin xyz=1.3877787807814456755e-17 0.078649999999999137268 0.036999999999999574896 rpy=3.141592653589793116 -5.3297228769912622595e-22 -2.2267995332275346432e-26 -> xyz=0 0.07865 0.0001 rpy=-0 -0 -1.5708; parent knee_and_ankle_assembly_3 -> right_cache
- joint trunk_frame: origin xyz=-0.024000000000000760308 -2.4112656316077618612e-16 0.088190938812376745704 rpy=-1.4062102177136726269e-16 -9.4252837597218562265e-17 7.8061435390716270015e-33 -> xyz=-0.024 -0 0.0881909 rpy=-0 -0 0
